Commit message: add utm

File: h4r_farmbot_descriptions/def/farmbot/utm.xacro (robot description, xacro)
@@ -4,5 +4,5 @@
        xmlns:interface="http://playerstage.sourceforge.net/gazebo/xmlschema/#interface"
        xmlns:xacro="http://ros.org/wiki/xacro">
-   <xacro:rr_joint_fixed parent="vertical" child="utm" origin_z="${-vertical_length/2}" />
+   <xacro:rr_joint_fixed parent="vertical" child="utm" origin_y="0.0465" origin_z="${-vertical_length/2+0.002}" origin_Y="${-rr_const_pi/2}" />
    <xacro:arg name="mesh_version" default="v1.2" />
 	<link name="utm">
@@ -14,5 +14,22 @@
 		<collision>
 			<geometry>
-				<cylinder length="0.1" radius="0.05" />
+				 <mesh filename="package://h4r_farmbot_descriptions/mesh/$(arg mesh_version)/utm.stl"/>
+			</geometry>
+		</collision>
+		<xacro:rr_inertia_cylinder_solid r="0.05" h="0.1" mass="0.25" >
+			<origin xyz="0 0 0" rpy="0 0 0" />
+		</xacro:rr_inertia_cylinder_solid>
+	</link>
+	<xacro:rr_joint_fixed parent="utm" child="utm_cover" origin_z="0.051" origin_P="${-rr_const_pi}" origin_Y="${-rr_const_pi}" />
+   	<link name="utm_cover">
+		<visual>
+			<geometry>
+				 <mesh filename="package://h4r_farmbot_descriptions/mesh/$(arg mesh_version)/utm_cover.stl"/>
+			</geometry>
+		</visual>
+		<collision>
+			<origin xyz="0 0 0.015" rpy="0 0 0" />
+			<geometry>
+				<cylinder length="0.032" radius="0.035" />
 			</geometry>
 		</collision>
