Commit message: add watertool with magnet plugin - not working!

File: h4r_farmbot_descriptions/def/farmbot/bed.xacro (robot description, xacro)
@@ -4,5 +4,10 @@
        xmlns:interface="http://playerstage.sourceforge.net/gazebo/xmlschema/#interface"
        xmlns:xacro="http://ros.org/wiki/xacro">
+       <link name="world"/>
        <link name="base_link" />
+       <joint name="fixed" type="fixed">
+        <parent link="world"/>
+        <child link="base_link"/>
+       </joint>
        <rr_joint_fixed parent="base_link" child="soil" origin_z="${soil_height/2}" />
        <xacro:rr_simple_box name="soil" x_size="${bed_length}" y_size="${bed_width}" z_size="${soil_height}" gazebo_material="H4R/Soil0" density="1400" />

File: h4r_farmbot_descriptions/def/farmbot/properties.xacro (robot description, xacro)
@@ -26,5 +26,5 @@
     <xacro:property name="boom_support_height"                 value="0.5" />
     <xacro:property name="vertical_length"                     value="1.01" />
-    <xacro:property name="vertical_length_offset_start"        value="0.28" />
+    <xacro:property name="vertical_length_offset_start"        value="0.40" />
     <xacro:property name="vertical_length_offset_end"          value="0.01" />
     <xacro:property name="vertical_axis_slider_offset"         value="-0.05" />

File: h4r_farmbot_descriptions/def/farmbot/utm.xacro (robot description, xacro)
@@ -4,4 +4,5 @@
        xmlns:interface="http://playerstage.sourceforge.net/gazebo/xmlschema/#interface"
        xmlns:xacro="http://ros.org/wiki/xacro">
+    <xacro:include filename="$(find h4r_farmbot_descriptions)/def/common/magnet_group.xacro"/>
     <xacro:rr_joint_fixed parent="vertical" child="utm" origin_y="0.0465" origin_z="${-vertical_length/2+0.002}" origin_Y="${-rr_const_pi/2}" />
     <link name="utm">
@@ -37,3 +38,4 @@
         </xacro:rr_inertia_cylinder_solid>
     </link>
+    <xacro:fb_utm_magnet_group name="utm" parent="utm" origin_z="0.0075" magnet_strength="50" />
 </robot>

File: h4r_farmbot_descriptions/def/farmbot/vertical.xacro (robot description, xacro)
@@ -10,10 +10,10 @@
                      child="vertical"
                      origin_x="${-(vertical_height/2+boom_slider_width/2)}"
-                      origin_y="${vertical_axis_slider_offset}"
+                     origin_y="${vertical_axis_slider_offset}"
                      origin_z="${vertical_length/2-vertical_length_offset_start}"
-                     effort="1000.0"
-                     lower ="0"
-                     upper="${vertical_length-vertical_length_offset_start-vertical_length_offset_end}"
-                     velocity="30"
+                     effort="30.0"
+                     lower ="${-(vertical_length-vertical_length_offset_start-vertical_length_offset_end)}"
+                     upper="0"
+                     velocity="0.5"
                      axis="z"
                      ros_control="${ros_control}"
