Commit message: spawn toolbay separately

File: h4r_farmbot_descriptions/def/farmbot/toolbays.xacro (robot description, xacro)
@@ -18,10 +18,10 @@
             <visual>
                 <geometry>
-                    <mesh filename="package://h4r_farmbot_descriptions/mesh/${mesh_version}/toolbay.stl"/>
+                    <mesh filename="package://h4r_farmbot_descriptions/mesh/${mesh_version}/toolbay_fancy.dae"/>
                 </geometry>
             </visual>
             <collision>
                 <geometry>
-                    <mesh filename="package://h4r_farmbot_descriptions/mesh/${mesh_version}/toolbay.stl"/>
+                    <mesh filename="package://h4r_farmbot_descriptions/mesh/${mesh_version}/toolbay_fancy.dae"/>
                 </geometry>
             </collision>
@@ -32,20 +32,20 @@
     </xacro:macro>
     <xacro:fb_toolbay
-           parent="rail_frame_2"
+           parent="base_link"
            number="0"
            mesh_version="${mesh_version}"
-           origin_z="0.113"
-           origin_y="-0.117"
-           origin_x="0.25"
-           origin_Y="${rr_const_pi}"
+           origin_z="${bed_height+foot_height+rail_height/2+0.113}"
+           origin_y="+0.25"
+           origin_x="${-bed_length/2+0.1}"
+           origin_Y="${-rr_const_pi/2}"
         />
     <xacro:fb_toolbay
-           parent="rail_frame_2"
+           parent="base_link"
            number="1"
            mesh_version="${mesh_version}"
-           origin_z="0.113"
-           origin_y="-0.117"
-           origin_x="-0.25"
-           origin_Y="${rr_const_pi}"
+           origin_z="${bed_height+foot_height+rail_height/2+0.113}"
+           origin_y="-0.25"
+           origin_x="${-bed_length/2+0.1}"
+           origin_Y="${-rr_const_pi/2}"
         />
 </robot>
