Commit message: copy and integrate examples from  gantry bot (rapid robot xacros)

File: h4r_farmbot_descriptions/def/farmbot.xacro (robot description, xacro)
@@ -5,5 +5,9 @@
        xmlns:xacro="http://ros.org/wiki/xacro">
        	<xacro:include filename="$(find h4r_rapid_robot_xacros)/def/rapid_robot.xacro"/>
-       	<xacro:include filename="$(find h4r_farmbot_descriptions)/def/farmbot/properties.xacro"/>
+        <xacro:include filename="$(find h4r_farmbot_descriptions)/def/farmbot/frame.xacro"/>
+        <xacro:include filename="$(find h4r_farmbot_descriptions)/def/farmbot/properties.xacro"/>
        	<xacro:include filename="$(find h4r_farmbot_descriptions)/def/farmbot/bed.xacro"/>
+        <xacro:include filename="$(find h4r_farmbot_descriptions)/def/farmbot/rails.xacro"/>
+        <xacro:include filename="$(find h4r_farmbot_descriptions)/def/farmbot/boom.xacro"/>
+       	<xacro:include filename="$(find h4r_farmbot_descriptions)/def/farmbot/vertical.xacro"/>
 </robot>

File: h4r_farmbot_descriptions/def/farmbot/bed.xacro (robot description, xacro)
@@ -7,41 +7,47 @@
        <rr_joint_fixed parent="base_link" child="soil" origin_z="${soil_height/2}" />
        <xacro:rr_simple_box name="soil" x_size="${bed_length}" y_size="${bed_width}" z_size="${soil_height}" gazebo_material="H4R/Soil0" density="1400" />
-       <xacro:macro name="fb_bed_side" params="side">
-       		<xacro:if value="${side==0 or side==1}">
-       			<xacro:property name="origin_x_abs" value="0"/>
-       			<xacro:property name="origin_y_abs" value="${bed_width/2+wood_board_width/2}"/>
-				<xacro:property name="length" value="${bed_length}"/>
-       			<xacro:property name="rot" value="0"/>
-       		</xacro:if>
-       		<xacro:if value="${side==2 or side==3}">
-       			<xacro:property name="origin_x_abs" value="${bed_length/2+wood_board_width/2}"/>
-       			<xacro:property name="origin_y_abs" value="0"/>
-				<xacro:property name="length" value="${bed_width+wood_board_width*2}"/>
-       			<xacro:property name="rot" value="${rr_const_pi/2}"/>
-       		</xacro:if>
-       		<xacro:if value="${side%2}">
-       			<xacro:property name="origin_x" value="${origin_x_abs}"/>
-       			<xacro:property name="origin_y" value="${origin_y_abs}"/>
-       		</xacro:if>
-       		<xacro:unless value="${side%2}">
-       			<xacro:property name="origin_x" value="${-origin_x_abs}"/>
-       			<xacro:property name="origin_y" value="${-origin_y_abs}"/>
-       		</xacro:unless>
-       		<rr_joint_fixed parent="base_link"
-       		                child="bed_wood_frame_${side}"
-       		                origin_x="${origin_x}"
-       		                origin_y="${origin_y}"
-       			            origin_z="${bed_height/2}"
-       		                origin_Y="${rot}"/>
-       		<xacro:rr_simple_box name="bed_wood_frame_${side}"
-       							 x_size="${length}"
-       							 y_size="${wood_board_width}"
-       							 z_size="${bed_height}"
-       							 gazebo_material="H4R/WoodFaded0"
-       							 density="730" />
-       </xacro:macro>
-       <xacro:fb_bed_side side="0"/>
-	   <xacro:fb_bed_side side="1"/>
-       <xacro:fb_bed_side side="2"/>
-       <xacro:fb_bed_side side="3"/>
+       <xacro:fb_frame
+	       name="bed_wood_frame"
+	       parent="base_link"
+	       side="0"
+	       width="${bed_width}"
+		   height="${bed_height}"
+       	   length="${bed_length}"
+	       thickness="0.04"
+	       gazebo_material="H4R/WoodFaded0"
+	       density="730"
+       	/>
+       	<xacro:fb_frame
+	       name="bed_wood_frame"
+	       parent="base_link"
+	       side="1"
+	       width="${bed_width}"
+		   height="${bed_height}"
+       	   length="${bed_length}"
+	       thickness="0.04"
+	       gazebo_material="H4R/WoodFaded0"
+	       density="730"
+       	/>
+       	<xacro:fb_frame
+	       name="bed_wood_frame"
+	       parent="base_link"
+	       side="2"
+	       width="${bed_width}"
+		   height="${bed_height}"
+       	   length="${bed_length}"
+	       thickness="0.04"
+	       gazebo_material="H4R/WoodFaded0"
+	       density="730"
+       	/>
+        <xacro:fb_frame
+	       name="bed_wood_frame"
+	       parent="base_link"
+	       side="3"
+	       width="${bed_width}"
+		   height="${bed_height}"
+       	   length="${bed_length}"
+	       thickness="0.04"
+	       gazebo_material="H4R/WoodFaded0"
+	       density="730"
+       	/>
 </robot>

File: h4r_farmbot_descriptions/def/farmbot/properties.xacro (robot description, xacro)
@@ -4,8 +4,57 @@
        xmlns:interface="http://playerstage.sourceforge.net/gazebo/xmlschema/#interface"
        xmlns:xacro="http://ros.org/wiki/xacro">
-       <xacro:property name="bed_height"  value="1.0" />
-       <xacro:property name="bed_length"  value="5.0" />
-       <xacro:property name="bed_width"   value="2.0" />
-       <xacro:property name="soil_height" value="0.9" />
-       <xacro:property name="wood_board_width"  value="0.04" />
+		<xacro:property name="bed_height"  value="1.0" />
+		<xacro:property name="bed_length"  value="5.0" />
+		<xacro:property name="bed_width"   value="2.0" />
+		<xacro:property name="soil_height" value="0.9" />
+		<xacro:property name="wood_board_width"  value="0.04" />
+		<xacro:property name="vslot2020_weight_per_meter" value="0.75" />
+		<xacro:property name="vslot2020_height"   		value="0.02" />
+		<xacro:property name="vslot2020_width"   		value="0.02" />
+		<xacro:property name="vslot2040_weight_per_meter" value="0.85" />
+		<xacro:property name="vslot2040_height"   		value="0.04" />
+		<xacro:property name="vslot2040_width"   		value="0.02" />
+		<xacro:property name="vslot2060_weight_per_meter" value="1.5" />
+		<xacro:property name="vslot2060_height"   		value="0.06" />
+		<xacro:property name="vslot2060_width"   		value="0.02" />
+		<xacro:property name="rail_length"  		value="${bed_length}" />
+		<xacro:property name="rail_length_offset_start"  		value="0.01" />
+		<xacro:property name="rail_length_offset_end"  			value="0.01" />
+		<xacro:property name="boom_length"  					value="${bed_width+rail_width*2+wood_board_width}" />
+		<xacro:property name="boom_length_offset_start"  		value="0.01" />
+		<xacro:property name="boom_length_offset_end"  			value="0.01" />
+		<xacro:property name="boom_support_height"  value="0.5" />
+		<xacro:property name="vertical_length"  	value="1.01" />
+		<xacro:property name="vertical_length_offset_start"  	value="0.28" />
+		<xacro:property name="vertical_length_offset_end"  		value="0.01" />
+		<xacro:property name="vertical_axis_slider_offset"  value="-0.05" />
+		<xacro:property name="rail_width"   		value="${vslot2040_width}" />
+		<xacro:property name="rail_height"  		value="${vslot2040_height}" />
+		<xacro:property name="rail_weight"  		value="${rail_length*vslot2040_weight_per_meter}" />
+		<xacro:property name="rail_end_width"   	value="${rail_width}" />
+		<xacro:property name="rail_end_height"  	value="${rail_height}" />
+		<xacro:property name="rail_end_length"  	value="${boom_length}" />
+		<xacro:property name="rail_end_weight"  	value="${rail_end_length*vslot2040_weight_per_meter}" />
+		<xacro:property name="boom_support_length" value="${vslot2060_height}" />
+		<xacro:property name="boom_support_width"  value="${vslot2060_width}" />
+		<xacro:property name="boom_support_weight" value="${boom_support_height*vslot2060_weight_per_meter}" />
+		<xacro:property name="rail_slider_width"   	value="0.02" />
+		<xacro:property name="rail_slider_length"   value="${boom_support_length+0.02}" />
+		<xacro:property name="rail_slider_height"   value="${rail_height+0.04}" />
+		<xacro:property name="rail_slider_weight"   value="1.0" />
+		<xacro:property name="boom_width"   		value="${vslot2060_width}" />
+		<xacro:property name="boom_height"  		value="${vslot2060_height}" />
+		<xacro:property name="boom_weight"  		value="${boom_length*vslot2060_weight_per_meter}" />
+		<xacro:property name="boom_slider_length"  	value="0.17" />
+		<xacro:property name="boom_slider_width"   	value="0.01" />
+		<xacro:property name="boom_slider_height"  	value="0.15" />
+		<xacro:property name="boom_slider_weight"  	value="1.0" />
+		<xacro:property name="vertical_width"   	value="${vslot2020_height}" />
+		<xacro:property name="vertical_height"  	value="${vslot2020_width}" />
+		<xacro:property name="vertical_weight"  	value="${vertical_length*vslot2020_weight_per_meter}" />
+		<xacro:property name="foot_length"  	value="0.1" />
+		<xacro:property name="foot_width"   	value="0.05" />
+		<xacro:property name="foot_height"  	value="0.05" />
+		<xacro:property name="foot_weight"  	value="1.0" />
+		<xacro:property name="ros_control"  	value="true" />
 </robot>

Commit message: add toolbays

File: h4r_farmbot_descriptions/def/farmbot.xacro (robot description, xacro)
@@ -12,3 +12,4 @@
        	<xacro:include filename="$(find h4r_farmbot_descriptions)/def/farmbot/vertical.xacro"/>
        	<xacro:include filename="$(find h4r_farmbot_descriptions)/def/farmbot/utm.xacro"/>
+       	<xacro:include filename="$(find h4r_farmbot_descriptions)/def/farmbot/toolbays.xacro"/>
 </robot>

File: h4r_farmbot_descriptions/def/farmbot/properties.xacro (robot description, xacro)
@@ -58,3 +58,4 @@
 		<xacro:property name="foot_weight"  	value="1.0" />
 		<xacro:property name="ros_control"  	value="true" />
+       	<xacro:property name="mesh_version"  	value="v1.2" />
 </robot>

File: h4r_farmbot_descriptions/def/farmbot/utm.xacro (robot description, xacro)
@@ -5,14 +5,13 @@
        xmlns:xacro="http://ros.org/wiki/xacro">
    <xacro:rr_joint_fixed parent="vertical" child="utm" origin_y="0.0465" origin_z="${-vertical_length/2+0.002}" origin_Y="${-rr_const_pi/2}" />
-   <xacro:arg name="mesh_version" default="v1.2" />
 	<link name="utm">
 		<visual>
 			<geometry>
-				 <mesh filename="package://h4r_farmbot_descriptions/mesh/$(arg mesh_version)/utm.stl"/>
+				 <mesh filename="package://h4r_farmbot_descriptions/mesh/${mesh_version}/utm.stl"/>
 			</geometry>
 		</visual>
 		<collision>
 			<geometry>
-				 <mesh filename="package://h4r_farmbot_descriptions/mesh/$(arg mesh_version)/utm.stl"/>
+				 <mesh filename="package://h4r_farmbot_descriptions/mesh/${mesh_version}/utm.stl"/>
 			</geometry>
 		</collision>
@@ -25,5 +24,5 @@
 		<visual>
 			<geometry>
-				 <mesh filename="package://h4r_farmbot_descriptions/mesh/$(arg mesh_version)/utm_cover.stl"/>
+				 <mesh filename="package://h4r_farmbot_descriptions/mesh/${mesh_version}/utm_cover.stl"/>
 			</geometry>
 		</visual>
