Commit message: reformat and add roscontrol plugin

File: h4r_farmbot_descriptions/def/farmbot.xacro (robot description, xacro)
@@ -3,13 +3,17 @@
        xmlns:controller="http://playerstage.sourceforge.net/gazebo/xmlschema/#controller"
        xmlns:interface="http://playerstage.sourceforge.net/gazebo/xmlschema/#interface"
-       xmlns:xacro="http://ros.org/wiki/xacro">
-       	<xacro:include filename="$(find h4r_rapid_robot_xacros)/def/rapid_robot.xacro"/>
-        <xacro:include filename="$(find h4r_farmbot_descriptions)/def/farmbot/frame.xacro"/>
-        <xacro:include filename="$(find h4r_farmbot_descriptions)/def/farmbot/properties.xacro"/>
-       	<xacro:include filename="$(find h4r_farmbot_descriptions)/def/farmbot/bed.xacro"/>
-        <xacro:include filename="$(find h4r_farmbot_descriptions)/def/farmbot/rails.xacro"/>
-        <xacro:include filename="$(find h4r_farmbot_descriptions)/def/farmbot/boom.xacro"/>
-       	<xacro:include filename="$(find h4r_farmbot_descriptions)/def/farmbot/vertical.xacro"/>
-       	<xacro:include filename="$(find h4r_farmbot_descriptions)/def/farmbot/utm.xacro"/>
-       	<xacro:include filename="$(find h4r_farmbot_descriptions)/def/farmbot/toolbays.xacro"/>
+       xmlns:xacro="http://ros.org/wiki/xacro" name="h4r_farmbot">
+    <xacro:include filename="$(find h4r_rapid_robot_xacros)/def/rapid_robot.xacro"/>
+    <xacro:include filename="$(find h4r_farmbot_descriptions)/def/farmbot/frame.xacro"/>
+    <xacro:include filename="$(find h4r_farmbot_descriptions)/def/farmbot/properties.xacro"/>
+    <xacro:include filename="$(find h4r_farmbot_descriptions)/def/farmbot/bed.xacro"/>
+    <xacro:include filename="$(find h4r_farmbot_descriptions)/def/farmbot/rails.xacro"/>
+    <!--
+    <xacro:include filename="$(find h4r_farmbot_descriptions)/def/farmbot/boom.xacro"/>
+    <xacro:include filename="$(find h4r_farmbot_descriptions)/def/farmbot/vertical.xacro"/>
+    <xacro:include filename="$(find h4r_farmbot_descriptions)/def/farmbot/utm.xacro"/>
+    <xacro:include filename="$(find h4r_farmbot_descriptions)/def/farmbot/toolbays.xacro"/>
+    -->
+    <!-- ROS CONTROL PLUGIN -->
+    <xacro:rr_roscontrol_controller />
 </robot>

File: h4r_farmbot_descriptions/def/farmbot/bed.xacro (robot description, xacro)
@@ -8,46 +8,46 @@
        <xacro:rr_simple_box name="soil" x_size="${bed_length}" y_size="${bed_width}" z_size="${soil_height}" gazebo_material="H4R/Soil0" density="1400" />
        <xacro:fb_frame
-	       name="bed_wood_frame"
-	       parent="base_link"
-	       side="0"
-	       width="${bed_width}"
-		   height="${bed_height}"
-       	   length="${bed_length}"
-	       thickness="0.04"
-	       gazebo_material="H4R/WoodFaded0"
-	       density="730"
-       	/>
-       	<xacro:fb_frame
-	       name="bed_wood_frame"
-	       parent="base_link"
-	       side="1"
-	       width="${bed_width}"
-		   height="${bed_height}"
-       	   length="${bed_length}"
-	       thickness="0.04"
-	       gazebo_material="H4R/WoodFaded0"
-	       density="730"
-       	/>
-       	<xacro:fb_frame
-	       name="bed_wood_frame"
-	       parent="base_link"
-	       side="2"
-	       width="${bed_width}"
-		   height="${bed_height}"
-       	   length="${bed_length}"
-	       thickness="0.04"
-	       gazebo_material="H4R/WoodFaded0"
-	       density="730"
-       	/>
+           name="bed_wood_frame"
+           parent="base_link"
+           side="0"
+           width="${bed_width}"
+           height="${bed_height}"
+              length="${bed_length}"
+           thickness="0.04"
+           gazebo_material="H4R/WoodFaded0"
+           density="730"
+           />
+           <xacro:fb_frame
+           name="bed_wood_frame"
+           parent="base_link"
+           side="1"
+           width="${bed_width}"
+           height="${bed_height}"
+              length="${bed_length}"
+           thickness="0.04"
+           gazebo_material="H4R/WoodFaded0"
+           density="730"
+           />
+           <xacro:fb_frame
+           name="bed_wood_frame"
+           parent="base_link"
+           side="2"
+           width="${bed_width}"
+           height="${bed_height}"
+              length="${bed_length}"
+           thickness="0.04"
+           gazebo_material="H4R/WoodFaded0"
+           density="730"
+           />
         <xacro:fb_frame
-	       name="bed_wood_frame"
-	       parent="base_link"
-	       side="3"
-	       width="${bed_width}"
-		   height="${bed_height}"
-       	   length="${bed_length}"
-	       thickness="0.04"
-	       gazebo_material="H4R/WoodFaded0"
-	       density="730"
-       	/>
+           name="bed_wood_frame"
+           parent="base_link"
+           side="3"
+           width="${bed_width}"
+           height="${bed_height}"
+              length="${bed_length}"
+           thickness="0.04"
+           gazebo_material="H4R/WoodFaded0"
+           density="730"
+           />
 </robot>

File: h4r_farmbot_descriptions/def/farmbot/boom.xacro (robot description, xacro)
@@ -4,35 +4,35 @@
        xmlns:interface="http://playerstage.sourceforge.net/gazebo/xmlschema/#interface"
        xmlns:xacro="http://ros.org/wiki/xacro">
-<!-- Boom Supports -->
-<xacro:rr_simple_box name="boom_support_left"  x_size="${boom_support_length}" y_size="${boom_support_width}" z_size="${boom_support_height}" weight="${boom_support_weight}" gazebo_material="Gazebo/FlatBlack" />
-<xacro:rr_simple_box name="boom_support_right" x_size="${boom_support_length}" y_size="${boom_support_width}" z_size="${boom_support_height}" weight="${boom_support_weight}" gazebo_material="Gazebo/FlatBlack" />
-<xacro:property name="boom_support_y_pos"   	value="${rail_slider_width/2+boom_support_width/2}" />
-<xacro:property name="boom_support_z_pos"   	value="${boom_support_height/2+rail_height/2}" />
-<xacro:rr_joint_fixed parent="rail_slider_left" child="boom_support_left"
-					  origin_y="${boom_support_y_pos}"
-   					  origin_z="${boom_support_z_pos}" />
-<xacro:rr_joint_fixed parent="rail_slider_right" child="boom_support_right"
-					  origin_y="${-boom_support_y_pos}"
-   					  origin_z="${boom_support_z_pos}" />
-<!-- Boom -->
-<xacro:rr_simple_box name="boom" x_size="${boom_width}" y_size="${boom_length}" z_size="${boom_height}" weight="${boom_weight}" gazebo_material="Gazebo/FlatBlack"  />
-<xacro:rr_joint_fixed parent="boom_support_left" child="boom"
-					  origin_x="${-(boom_support_length/2-boom_width/2)}"
-					  origin_y="${boom_length/2-boom_support_width/2}"
-   					  origin_z="${boom_support_height/2+boom_height/2}"/>
-<!-- Boom Axis -->
-       <xacro:rr_simple_box name="boom_slider"  x_size="${boom_slider_width}" y_size="${boom_slider_length}" z_size="${boom_slider_height}" weight="${boom_slider_weight}" gazebo_material="Gazebo/FlatBlack" />
-	   <xacro:rr_linear_axis parent="boom"
-	                         child="boom_slider"
-	   						 origin_x="${-(boom_slider_width/2+boom_width/2)}"
-							 origin_y="${(boom_length-boom_slider_length)/2+boom_length_offset_start}"
-	   						 effort="1000.0"
-							 lower ="0"
-							 upper="${boom_length-boom_slider_length-boom_length_offset_start-boom_length_offset_end}"
-							 velocity="30"
-							 axis="y"
-	   						 ros_control="${ros_control}"
-	   						 ros_control_position="true"
-	   						 joint_name="boom_joint"
-   						/>
+    <!-- Boom Supports -->
+    <xacro:rr_simple_box name="boom_support_left"  x_size="${boom_support_length}" y_size="${boom_support_width}" z_size="${boom_support_height}" weight="${boom_support_weight}" gazebo_material="Gazebo/FlatBlack" />
+    <xacro:rr_simple_box name="boom_support_right" x_size="${boom_support_length}" y_size="${boom_support_width}" z_size="${boom_support_height}" weight="${boom_support_weight}" gazebo_material="Gazebo/FlatBlack" />
+    <xacro:property name="boom_support_y_pos"       value="${rail_slider_width/2+boom_support_width/2}" />
+    <xacro:property name="boom_support_z_pos"       value="${boom_support_height/2+rail_height/2}" />
+    <xacro:rr_joint_fixed parent="rail_slider_left" child="boom_support_left"
+                      origin_y="${boom_support_y_pos}"
+                      origin_z="${boom_support_z_pos}" />
+    <xacro:rr_joint_fixed parent="rail_slider_right" child="boom_support_right"
+                      origin_y="${-boom_support_y_pos}"
+                      origin_z="${boom_support_z_pos}" />
+    <!-- Boom -->
+    <xacro:rr_simple_box name="boom" x_size="${boom_width}" y_size="${boom_length}" z_size="${boom_height}" weight="${boom_weight}" gazebo_material="Gazebo/FlatBlack"  />
+    <xacro:rr_joint_fixed parent="boom_support_left" child="boom"
+                      origin_x="${-(boom_support_length/2-boom_width/2)}"
+                      origin_y="${boom_length/2-boom_support_width/2}"
+                      origin_z="${boom_support_height/2+boom_height/2}"/>
+    <!-- Boom Axis -->
+    <xacro:rr_simple_box name="boom_slider"  x_size="${boom_slider_width}" y_size="${boom_slider_length}" z_size="${boom_slider_height}" weight="${boom_slider_weight}" gazebo_material="Gazebo/FlatBlack" />
+    <xacro:rr_linear_axis parent="boom"
+                             child="boom_slider"
+                             origin_x="${-(boom_slider_width/2+boom_width/2)}"
+                             origin_y="${(boom_length-boom_slider_length)/2+boom_length_offset_start}"
+                             effort="1000.0"
+                             lower ="0"
+                             upper="${boom_length-boom_slider_length-boom_length_offset_start-boom_length_offset_end}"
+                             velocity="30"
+                             axis="y"
+                             ros_control="${ros_control}"
+                             ros_control_position="true"
+                             joint_name="boom_joint"
+                           />
 </robot>

File: h4r_farmbot_descriptions/def/farmbot/frame.xacro (robot description, xacro)
@@ -5,36 +5,36 @@
        xmlns:xacro="http://ros.org/wiki/xacro">
 <xacro:macro name="fb_frame" params="name parent side width length thickness height height_offset:=0 gazebo_material:=Gazebo/Grey density:=1" >
-       		<xacro:if value="${side==0 or side==1}">
-       			<xacro:property name="origin_x_abs" value="0"/>
-       			<xacro:property name="origin_y_abs" value="${width/2+thickness/2}"/>
-				<xacro:property name="bar_length" value="${length}"/>
-       			<xacro:property name="rot" value="0"/>
-       		</xacro:if>
-       		<xacro:if value="${side==2 or side==3}">
-       			<xacro:property name="origin_x_abs" value="${length/2+thickness/2}"/>
-       			<xacro:property name="origin_y_abs" value="0"/>
-				<xacro:property name="bar_length" value="${width+thickness*2}"/>
-       			<xacro:property name="rot" value="${rr_const_pi/2}"/>
-       		</xacro:if>
-       		<xacro:if value="${side%2}">
-       			<xacro:property name="origin_x" value="${origin_x_abs}"/>
-       			<xacro:property name="origin_y" value="${origin_y_abs}"/>
-       		</xacro:if>
-       		<xacro:unless value="${side%2}">
-       			<xacro:property name="origin_x" value="${-origin_x_abs}"/>
-       			<xacro:property name="origin_y" value="${-origin_y_abs}"/>
-       		</xacro:unless>
-       		<rr_joint_fixed parent="${parent}"
-       		                child="${name}_${side}"
-       		                origin_x="${origin_x}"
-       		                origin_y="${origin_y}"
-       			            origin_z="${height/2+height_offset}"
-       		                origin_Y="${rot}"/>
-       		<xacro:rr_simple_box name="${name}_${side}"
-       							 x_size="${bar_length}"
-       							 y_size="${thickness}"
-       							 z_size="${height}"
-       							 gazebo_material="${gazebo_material}"
-       							 density="${density}" />
+               <xacro:if value="${side==0 or side==1}">
+                   <xacro:property name="origin_x_abs" value="0"/>
+                   <xacro:property name="origin_y_abs" value="${width/2+thickness/2}"/>
+                <xacro:property name="bar_length" value="${length}"/>
+                   <xacro:property name="rot" value="0"/>
+               </xacro:if>
+               <xacro:if value="${side==2 or side==3}">
+                   <xacro:property name="origin_x_abs" value="${length/2+thickness/2}"/>
+                   <xacro:property name="origin_y_abs" value="0"/>
+                <xacro:property name="bar_length" value="${width+thickness*2}"/>
+                   <xacro:property name="rot" value="${rr_const_pi/2}"/>
+               </xacro:if>
+               <xacro:if value="${side%2}">
+                   <xacro:property name="origin_x" value="${origin_x_abs}"/>
+                   <xacro:property name="origin_y" value="${origin_y_abs}"/>
+               </xacro:if>
+               <xacro:unless value="${side%2}">
+                   <xacro:property name="origin_x" value="${-origin_x_abs}"/>
+                   <xacro:property name="origin_y" value="${-origin_y_abs}"/>
+               </xacro:unless>
+               <rr_joint_fixed parent="${parent}"
+                               child="${name}_${side}"
+                               origin_x="${origin_x}"
+                               origin_y="${origin_y}"
+                               origin_z="${height/2+height_offset}"
+                               origin_Y="${rot}"/>
+               <xacro:rr_simple_box name="${name}_${side}"
+                                    x_size="${bar_length}"
+                                    y_size="${thickness}"
+                                    z_size="${height}"
+                                    gazebo_material="${gazebo_material}"
+                                    density="${density}" />
        </xacro:macro>
 </robot>

File: h4r_farmbot_descriptions/def/farmbot/properties.xacro (robot description, xacro)
@@ -4,58 +4,58 @@
        xmlns:interface="http://playerstage.sourceforge.net/gazebo/xmlschema/#interface"
        xmlns:xacro="http://ros.org/wiki/xacro">
-		<xacro:property name="bed_height"  value="1.0" />
-		<xacro:property name="bed_length"  value="5.0" />
-		<xacro:property name="bed_width"   value="2.0" />
-		<xacro:property name="soil_height" value="0.9" />
-		<xacro:property name="wood_board_width"  value="0.04" />
-		<xacro:property name="vslot2020_weight_per_meter" value="0.75" />
-		<xacro:property name="vslot2020_height"   		value="0.02" />
-		<xacro:property name="vslot2020_width"   		value="0.02" />
-		<xacro:property name="vslot2040_weight_per_meter" value="0.85" />
-		<xacro:property name="vslot2040_height"   		value="0.04" />
-		<xacro:property name="vslot2040_width"   		value="0.02" />
-		<xacro:property name="vslot2060_weight_per_meter" value="1.5" />
-		<xacro:property name="vslot2060_height"   		value="0.06" />
-		<xacro:property name="vslot2060_width"   		value="0.02" />
-		<xacro:property name="rail_length"  		value="${bed_length}" />
-		<xacro:property name="rail_length_offset_start"  		value="0.01" />
-		<xacro:property name="rail_length_offset_end"  			value="0.01" />
-		<xacro:property name="boom_length"  					value="${bed_width+rail_width*2+wood_board_width}" />
-		<xacro:property name="boom_length_offset_start"  		value="0.01" />
-		<xacro:property name="boom_length_offset_end"  			value="0.01" />
-		<xacro:property name="boom_support_height"  value="0.5" />
-		<xacro:property name="vertical_length"  	value="1.01" />
-		<xacro:property name="vertical_length_offset_start"  	value="0.28" />
-		<xacro:property name="vertical_length_offset_end"  		value="0.01" />
-		<xacro:property name="vertical_axis_slider_offset"  value="-0.05" />
-		<xacro:property name="rail_width"   		value="${vslot2040_width}" />
-		<xacro:property name="rail_height"  		value="${vslot2040_height}" />
-		<xacro:property name="rail_weight"  		value="${rail_length*vslot2040_weight_per_meter}" />
-		<xacro:property name="rail_end_width"   	value="${rail_width}" />
-		<xacro:property name="rail_end_height"  	value="${rail_height}" />
-		<xacro:property name="rail_end_length"  	value="${boom_length}" />
-		<xacro:property name="rail_end_weight"  	value="${rail_end_length*vslot2040_weight_per_meter}" />
-		<xacro:property name="boom_support_length" value="${vslot2060_height}" />
-		<xacro:property name="boom_support_width"  value="${vslot2060_width}" />
-		<xacro:property name="boom_support_weight" value="${boom_support_height*vslot2060_weight_per_meter}" />
-		<xacro:property name="rail_slider_width"   	value="0.02" />
-		<xacro:property name="rail_slider_length"   value="${boom_support_length+0.02}" />
-		<xacro:property name="rail_slider_height"   value="${rail_height+0.04}" />
-		<xacro:property name="rail_slider_weight"   value="1.0" />
-		<xacro:property name="boom_width"   		value="${vslot2060_width}" />
-		<xacro:property name="boom_height"  		value="${vslot2060_height}" />
-		<xacro:property name="boom_weight"  		value="${boom_length*vslot2060_weight_per_meter}" />
-		<xacro:property name="boom_slider_length"  	value="0.17" />
-		<xacro:property name="boom_slider_width"   	value="0.01" />
-		<xacro:property name="boom_slider_height"  	value="0.15" />
-		<xacro:property name="boom_slider_weight"  	value="1.0" />
-		<xacro:property name="vertical_width"   	value="${vslot2020_height}" />
-		<xacro:property name="vertical_height"  	value="${vslot2020_width}" />
-		<xacro:property name="vertical_weight"  	value="${vertical_length*vslot2020_weight_per_meter}" />
-		<xacro:property name="foot_length"  	value="0.1" />
-		<xacro:property name="foot_width"   	value="0.05" />
-		<xacro:property name="foot_height"  	value="0.05" />
-		<xacro:property name="foot_weight"  	value="1.0" />
-		<xacro:property name="ros_control"  	value="true" />
-       	<xacro:property name="mesh_version"  	value="v1.2" />
+    <xacro:property name="bed_height"                 value="1.0" />
+    <xacro:property name="bed_length"                 value="5.0" />
+    <xacro:property name="bed_width"                  value="2.0" />
+    <xacro:property name="soil_height"                value="0.9" />
+    <xacro:property name="wood_board_width"           value="0.04" />
+    <xacro:property name="vslot2020_weight_per_meter" value="0.75" />
+    <xacro:property name="vslot2020_height"           value="0.02" />
+    <xacro:property name="vslot2020_width"            value="0.02" />
+    <xacro:property name="vslot2040_weight_per_meter" value="0.85" />
+    <xacro:property name="vslot2040_height"           value="0.04" />
+    <xacro:property name="vslot2040_width"            value="0.02" />
+    <xacro:property name="vslot2060_weight_per_meter" value="1.5" />
+    <xacro:property name="vslot2060_height"           value="0.06" />
+    <xacro:property name="vslot2060_width"            value="0.02" />
+    <xacro:property name="rail_length"                         value="${bed_length}" />
+    <xacro:property name="rail_length_offset_start"            value="0.01" />
+    <xacro:property name="rail_length_offset_end"              value="0.01" />
+    <xacro:property name="boom_length"                         value="${bed_width+rail_width*2+wood_board_width}" />
+    <xacro:property name="boom_length_offset_start"            value="0.01" />
+    <xacro:property name="boom_length_offset_end"              value="0.01" />
+    <xacro:property name="boom_support_height"                 value="0.5" />
+    <xacro:property name="vertical_length"                     value="1.01" />
+    <xacro:property name="vertical_length_offset_start"        value="0.28" />
+    <xacro:property name="vertical_length_offset_end"          value="0.01" />
+    <xacro:property name="vertical_axis_slider_offset"         value="-0.05" />
+    <xacro:property name="rail_width"              value="${vslot2040_width}" />
+    <xacro:property name="rail_height"             value="${vslot2040_height}" />
+    <xacro:property name="rail_weight"             value="${rail_length*vslot2040_weight_per_meter}" />
+    <xacro:property name="rail_end_width"          value="${rail_width}" />
+    <xacro:property name="rail_end_height"         value="${rail_height}" />
+    <xacro:property name="rail_end_length"         value="${boom_length}" />
+    <xacro:property name="rail_end_weight"         value="${rail_end_length*vslot2040_weight_per_meter}" />
+    <xacro:property name="boom_support_length"     value="${vslot2060_height}" />
+    <xacro:property name="boom_support_width"      value="${vslot2060_width}" />
+    <xacro:property name="boom_support_weight"     value="${boom_support_height*vslot2060_weight_per_meter}" />
+    <xacro:property name="rail_slider_width"       value="0.02" />
+    <xacro:property name="rail_slider_length"      value="${boom_support_length+0.02}" />
+    <xacro:property name="rail_slider_height"      value="${rail_height+0.04}" />
+    <xacro:property name="rail_slider_weight"      value="1.0" />
+    <xacro:property name="boom_width"              value="${vslot2060_width}" />
+    <xacro:property name="boom_height"             value="${vslot2060_height}" />
+    <xacro:property name="boom_weight"             value="${boom_length*vslot2060_weight_per_meter}" />
+    <xacro:property name="boom_slider_length"      value="0.17" />
+    <xacro:property name="boom_slider_width"       value="0.01" />
+    <xacro:property name="boom_slider_height"      value="0.15" />
+    <xacro:property name="boom_slider_weight"      value="1.0" />
+    <xacro:property name="vertical_width"          value="${vslot2020_height}" />
+    <xacro:property name="vertical_height"         value="${vslot2020_width}" />
+    <xacro:property name="vertical_weight"         value="${vertical_length*vslot2020_weight_per_meter}" />
+    <xacro:property name="foot_length"             value="0.1" />
+    <xacro:property name="foot_width"              value="0.05" />
+    <xacro:property name="foot_height"             value="0.05" />
+    <xacro:property name="foot_weight"             value="1.0" />
+    <xacro:property name="ros_control"             value="true" />
+    <xacro:property name="mesh_version"            value="v1.2" />
 </robot>
