Commit message: reformat and add roscontrol plugin

File: h4r_farmbot_descriptions/def/farmbot/rails.xacro (robot description, xacro)
@@ -4,69 +4,70 @@
        xmlns:interface="http://playerstage.sourceforge.net/gazebo/xmlschema/#interface"
        xmlns:xacro="http://ros.org/wiki/xacro">
-       <xacro:fb_frame
-	       name="rail_frame"
-	       parent="base_link"
-	       side="0"
-	       width="${bed_width}"
-		   height="${rail_height}"
-		   height_offset="${bed_height+foot_height}"
-       	   length="${bed_length}"
-	       thickness="${rail_width}"
-	       gazebo_material="Gazebo/FlatBlack"
-	       density="730"
-       	/>
-       	<xacro:fb_frame
-	       name="rail_frame"
-	       parent="base_link"
-	       side="1"
-	       width="${bed_width}"
-		   height="${rail_height}"
-		   height_offset="${bed_height+foot_height}"
-       	   length="${bed_length}"
-	       thickness="${rail_width}"
-	       gazebo_material="Gazebo/FlatBlack"
-	       density="730"
-       	/>
-       	<xacro:fb_frame
-	       name="rail_frame"
-	       parent="base_link"
-	       side="2"
-	       width="${bed_width}"
-		   height="${rail_height}"
-		   height_offset="${bed_height+foot_height}"
-       	   length="${bed_length}"
-	       thickness="${rail_width}"
-	       gazebo_material="Gazebo/FlatBlack"
-	       density="730"
-       	/>
-        <xacro:fb_frame
-	       name="rail_frame"
-	       parent="base_link"
-	       side="3"
-	       width="${bed_width}"
-		   height="${rail_height}"
-		   height_offset="${bed_height+foot_height}"
-       	   length="${bed_length}"
-	       thickness="${rail_width}"
-	       gazebo_material="Gazebo/FlatBlack"
-	       density="730"
-       	/>
-       <!-- Rail Sliders -->
-	   <xacro:rr_simple_box name="rail_slider_left"  x_size="${rail_slider_length}" y_size="${rail_slider_width}" z_size="${rail_slider_height}" weight="${rail_slider_weight}" gazebo_material="Gazebo/FlatBlack" />
-	   <xacro:rr_simple_box name="rail_slider_right" x_size="${rail_slider_length}" y_size="${rail_slider_width}" z_size="${rail_slider_height}" weight="${rail_slider_weight}" gazebo_material="Gazebo/FlatBlack" />
-	   <xacro:rr_joint_fixed parent="rail_slider_left" child="rail_slider_right" origin_y="${bed_width + rail_slider_width + rail_width*2}" />
-	   <!-- Rail Axis -->
-	   <xacro:rr_linear_axis parent="rail_frame_0"
-			                  child="rail_slider_left"
-			   	              origin_x="${ -( (rail_length/2) - (rail_slider_length/2) ) + rail_length_offset_start}"
-							  origin_y="${ -( (rail_width/2)  + (rail_slider_width/2) )}"
-			   				  effort="1000.0"
-						      lower ="0"
-						      upper="${rail_length - rail_slider_width - rail_length_offset_start - rail_length_offset_end}"
-							  velocity="1"
-							  axis="x"
-							  ros_control="${ros_control}"
-			   				  ros_control_position="true"
-							  joint_name="rail_joint"
-								/>
+    <xacro:fb_frame
+           name="rail_frame"
+           parent="base_link"
+           side="0"
+           width="${bed_width}"
+           height="${rail_height}"
+           height_offset="${bed_height+foot_height}"
+           length="${bed_length}"
+           thickness="${rail_width}"
+           gazebo_material="Gazebo/FlatBlack"
+           density="730"
+           />
+    <xacro:fb_frame
+           name="rail_frame"
+           parent="base_link"
+           side="1"
+           width="${bed_width}"
+           height="${rail_height}"
+           height_offset="${bed_height+foot_height}"
+           length="${bed_length}"
+           thickness="${rail_width}"
+           gazebo_material="Gazebo/FlatBlack"
+           density="730"
+           />
+    <xacro:fb_frame
+           name="rail_frame"
+           parent="base_link"
+           side="2"
+           width="${bed_width}"
+           height="${rail_height}"
+           height_offset="${bed_height+foot_height}"
+              length="${bed_length}"
+           thickness="${rail_width}"
+           gazebo_material="Gazebo/FlatBlack"
+           density="730"
+           />
+    <xacro:fb_frame
+           name="rail_frame"
+           parent="base_link"
+           side="3"
+           width="${bed_width}"
+           height="${rail_height}"
+           height_offset="${bed_height+foot_height}"
+           length="${bed_length}"
+           thickness="${rail_width}"
+           gazebo_material="Gazebo/FlatBlack"
+           density="730"
+           />
+    <!-- Rail Sliders -->
+    <xacro:rr_simple_box name="rail_slider_left"  x_size="${rail_slider_length}" y_size="${rail_slider_width}" z_size="${rail_slider_height}" weight="${rail_slider_weight}" gazebo_material="Gazebo/FlatBlack" />
+    <xacro:rr_simple_box name="rail_slider_right" x_size="${rail_slider_length}" y_size="${rail_slider_width}" z_size="${rail_slider_height}" weight="${rail_slider_weight}" gazebo_material="Gazebo/FlatBlack" />
+    <xacro:rr_joint_fixed parent="rail_slider_left" child="rail_slider_right" origin_y="${bed_width + rail_slider_width + rail_width*2}" />
+    <!-- Rail Axis -->
+    <xacro:rr_linear_axis
+              parent="rail_frame_0"
+              child="rail_slider_left"
+              origin_x="${ -( (rail_length/2) - (rail_slider_length/2) ) + rail_length_offset_start}"
+              origin_y="${ -( (rail_width/2)  + (rail_slider_width/2) )}"
+              effort="1000.0"
+              lower ="0"
+              upper="${rail_length - rail_slider_width - rail_length_offset_start - rail_length_offset_end}"
+              velocity="1"
+              axis="x"
+              ros_control="${ros_control}"
+              ros_control_position="true"
+              joint_name="rail_joint"
+              />
 </robot>

File: h4r_farmbot_descriptions/def/farmbot/toolbays.xacro (robot description, xacro)
@@ -4,46 +4,46 @@
        xmlns:interface="http://playerstage.sourceforge.net/gazebo/xmlschema/#interface"
        xmlns:xacro="http://ros.org/wiki/xacro">
-       <xacro:macro name="fb_toolbay" params="number parent mesh_version origin_x:=0 origin_y:=0 origin_z:=0 origin_R:=0 origin_P:=0 origin_Y:=0" >
-       		 <xacro:rr_joint_fixed
-       		 parent="${parent}"
-       		 child="toolbay${number}"
-       		 origin_x="${origin_x}"
-       		 origin_y="${origin_y}"
-       		 origin_z="${origin_z}"
-       		 origin_R="${origin_R}"
-       		 origin_P="${origin_P}"
-       		 origin_Y="${origin_Y}"
-       		 	/>
-			<link name="toolbay${number}">
-				<visual>
-					<geometry>
-						 <mesh filename="package://h4r_farmbot_descriptions/mesh/${mesh_version}/toolbay.stl"/>
-					</geometry>
-				</visual>
-				<collision>
-					<geometry>
-						 <mesh filename="package://h4r_farmbot_descriptions/mesh/${mesh_version}/toolbay.stl"/>
-					</geometry>
-				</collision>
-				<xacro:rr_inertia_cylinder_solid r="0.05" h="0.1" mass="0.25" >
-					<origin xyz="0 0 0" rpy="0 0 0" />
-				</xacro:rr_inertia_cylinder_solid>
-			</link>
-       </xacro:macro>
-	   <xacro:fb_toolbay
-		   parent="rail_frame_3"
-		   number="0"
-		   mesh_version="${mesh_version}"
-		   origin_z="0.113"
-	   	   origin_y="0.117"
-		   origin_x="0.25"
-	    />
-	    <xacro:fb_toolbay
-		   parent="rail_frame_3"
-		   number="1"
-		   mesh_version="${mesh_version}"
-		   origin_z="0.113"
-	   	   origin_y="0.117"
-		   origin_x="-0.25"
-	    />
+    <xacro:macro name="fb_toolbay" params="number parent mesh_version origin_x:=0 origin_y:=0 origin_z:=0 origin_R:=0 origin_P:=0 origin_Y:=0" >
+        <xacro:rr_joint_fixed
+                parent="${parent}"
+                child="toolbay${number}"
+                origin_x="${origin_x}"
+                origin_y="${origin_y}"
+                origin_z="${origin_z}"
+                origin_R="${origin_R}"
+                origin_P="${origin_P}"
+                origin_Y="${origin_Y}"
+                    />
+        <link name="toolbay${number}">
+            <visual>
+                <geometry>
+                    <mesh filename="package://h4r_farmbot_descriptions/mesh/${mesh_version}/toolbay.stl"/>
+                </geometry>
+            </visual>
+            <collision>
+                <geometry>
+                    <mesh filename="package://h4r_farmbot_descriptions/mesh/${mesh_version}/toolbay.stl"/>
+                </geometry>
+            </collision>
+            <xacro:rr_inertia_cylinder_solid r="0.05" h="0.1" mass="0.25" >
+                <origin xyz="0 0 0" rpy="0 0 0" />
+            </xacro:rr_inertia_cylinder_solid>
+        </link>
+    </xacro:macro>
+    <xacro:fb_toolbay
+           parent="rail_frame_3"
+           number="0"
+           mesh_version="${mesh_version}"
+           origin_z="0.113"
+              origin_y="0.117"
+           origin_x="0.25"
+        />
+    <xacro:fb_toolbay
+           parent="rail_frame_3"
+           number="1"
+           mesh_version="${mesh_version}"
+           origin_z="0.113"
+              origin_y="0.117"
+           origin_x="-0.25"
+        />
 </robot>

File: h4r_farmbot_descriptions/def/farmbot/utm.xacro (robot description, xacro)
@@ -4,36 +4,36 @@
        xmlns:interface="http://playerstage.sourceforge.net/gazebo/xmlschema/#interface"
        xmlns:xacro="http://ros.org/wiki/xacro">
-   <xacro:rr_joint_fixed parent="vertical" child="utm" origin_y="0.0465" origin_z="${-vertical_length/2+0.002}" origin_Y="${-rr_const_pi/2}" />
-	<link name="utm">
-		<visual>
-			<geometry>
-				 <mesh filename="package://h4r_farmbot_descriptions/mesh/${mesh_version}/utm.stl"/>
-			</geometry>
-		</visual>
-		<collision>
-			<geometry>
-				 <mesh filename="package://h4r_farmbot_descriptions/mesh/${mesh_version}/utm.stl"/>
-			</geometry>
-		</collision>
-		<xacro:rr_inertia_cylinder_solid r="0.05" h="0.1" mass="0.25" >
-			<origin xyz="0 0 0" rpy="0 0 0" />
-		</xacro:rr_inertia_cylinder_solid>
-	</link>
-	<xacro:rr_joint_fixed parent="utm" child="utm_cover" origin_z="0.051" origin_P="${-rr_const_pi}" origin_Y="${-rr_const_pi}" />
-   	<link name="utm_cover">
-		<visual>
-			<geometry>
-				 <mesh filename="package://h4r_farmbot_descriptions/mesh/${mesh_version}/utm_cover.stl"/>
-			</geometry>
-		</visual>
-		<collision>
-			<origin xyz="0 0 0.015" rpy="0 0 0" />
-			<geometry>
-				<cylinder length="0.032" radius="0.035" />
-			</geometry>
-		</collision>
-		<xacro:rr_inertia_cylinder_solid r="0.05" h="0.1" mass="0.25" >
-			<origin xyz="0 0 0" rpy="0 0 0" />
-		</xacro:rr_inertia_cylinder_solid>
-	</link>
+    <xacro:rr_joint_fixed parent="vertical" child="utm" origin_y="0.0465" origin_z="${-vertical_length/2+0.002}" origin_Y="${-rr_const_pi/2}" />
+    <link name="utm">
+        <visual>
+            <geometry>
+                <mesh filename="package://h4r_farmbot_descriptions/mesh/${mesh_version}/utm.stl"/>
+            </geometry>
+        </visual>
+        <collision>
+            <geometry>
+                <mesh filename="package://h4r_farmbot_descriptions/mesh/${mesh_version}/utm.stl"/>
+            </geometry>
+        </collision>
+        <xacro:rr_inertia_cylinder_solid r="0.05" h="0.1" mass="0.25" >
+            <origin xyz="0 0 0" rpy="0 0 0" />
+        </xacro:rr_inertia_cylinder_solid>
+    </link>
+    <xacro:rr_joint_fixed parent="utm" child="utm_cover" origin_z="0.051" origin_P="${-rr_const_pi}" origin_Y="${-rr_const_pi}" />
+    <link name="utm_cover">
+        <visual>
+            <geometry>
+                <mesh filename="package://h4r_farmbot_descriptions/mesh/${mesh_version}/utm_cover.stl"/>
+            </geometry>
+        </visual>
+        <collision>
+            <origin xyz="0 0 0.015" rpy="0 0 0" />
+            <geometry>
+                <cylinder length="0.032" radius="0.035" />
+            </geometry>
+        </collision>
+        <xacro:rr_inertia_cylinder_solid r="0.05" h="0.1" mass="0.25" >
+            <origin xyz="0 0 0" rpy="0 0 0" />
+        </xacro:rr_inertia_cylinder_solid>
+    </link>
 </robot>

File: h4r_farmbot_descriptions/def/farmbot/vertical.xacro (robot description, xacro)
@@ -4,20 +4,20 @@
        xmlns:interface="http://playerstage.sourceforge.net/gazebo/xmlschema/#interface"
        xmlns:xacro="http://ros.org/wiki/xacro">
-<!-- Vertical -->
-<xacro:rr_simple_box name="vertical" x_size="${vertical_height}" y_size="${vertical_width}" z_size="${vertical_length}" weight="${vertical_weight}" gazebo_material="Gazebo/FlatBlack"/>
-<!-- Vertical Axis -->
-<xacro:rr_linear_axis parent="boom_slider"
+    <!-- Vertical -->
+    <xacro:rr_simple_box name="vertical" x_size="${vertical_height}" y_size="${vertical_width}" z_size="${vertical_length}" weight="${vertical_weight}" gazebo_material="Gazebo/FlatBlack"/>
+    <!-- Vertical Axis -->
+    <xacro:rr_linear_axis parent="boom_slider"
                      child="vertical"
-					 origin_x="${-(vertical_height/2+boom_slider_width/2)}"
- 					 origin_y="${vertical_axis_slider_offset}"
-					 origin_z="${vertical_length/2-vertical_length_offset_start}"
-					 effort="1000.0"
-					 lower ="0"
-					 upper="${vertical_length-vertical_length_offset_start-vertical_length_offset_end}"
-					 velocity="30"
-					 axis="z"
-					 ros_control="${ros_control}"
-	   				 ros_control_position="true"
-					 joint_name="vertical_joint"
-					/>
+                     origin_x="${-(vertical_height/2+boom_slider_width/2)}"
+                      origin_y="${vertical_axis_slider_offset}"
+                     origin_z="${vertical_length/2-vertical_length_offset_start}"
+                     effort="1000.0"
+                     lower ="0"
+                     upper="${vertical_length-vertical_length_offset_start-vertical_length_offset_end}"
+                     velocity="30"
+                     axis="z"
+                     ros_control="${ros_control}"
+                     ros_control_position="true"
+                     joint_name="vertical_joint"
+                    />
 </robot>
