Commit message: fix watering nozzel collision

File: h4r_farmbot_descriptions/def/tools/watering_nozzle.xacro (robot description, xacro)
@@ -14,7 +14,19 @@
             </visual>
             <collision>
-                <origin xyz="0 0 ${0.035/4}" rpy="0 0 0" />
+                <origin xyz="0 0 0.006" rpy="0 0 0" />
                 <geometry>
-                     <cylinder radius="0.035" length="0.016" />
+                    <box size="0.063 0.07 0.0074" />
+                </geometry>
+            </collision>
+            <collision>
+                <origin xyz="0 0 0.0112" rpy="0 0 0" />
+                <geometry>
+                    <cylinder radius="0.035" length="0.002" />
+                </geometry>
+            </collision>
+            <collision>
+                <origin xyz="0 0 0.001" rpy="0 0 0" />
+                <geometry>
+                    <cylinder radius="0.035" length="0.002" />
                 </geometry>
             </collision>

Commit message: add macro for tool collision

File: h4r_farmbot_descriptions/def/tools/watering_nozzle.xacro (robot description, xacro)
@@ -6,4 +6,5 @@
         <xacro:include filename="$(find h4r_rapid_robot_xacros)/def/rapid_robot.xacro"/>
         <xacro:include filename="$(find h4r_farmbot_descriptions)/def/common/magnet_group.xacro"/>
+        <xacro:include filename="$(find h4r_farmbot_descriptions)/def/common/tool_collision.xacro"/>
         <xacro:property name="mesh_version"            value="v1.2" />
         <link name="watering_nozzle_top">
@@ -13,22 +14,5 @@
                 </geometry>
             </visual>
-            <collision>
-                <origin xyz="0 0 0.006" rpy="0 0 0" />
-                <geometry>
-                    <box size="0.063 0.04 0.0074" />
-                </geometry>
-            </collision>
-            <collision>
-                <origin xyz="0 0 0.0112" rpy="0 0 0" />
-                <geometry>
-                    <cylinder radius="0.035" length="0.002" />
-                </geometry>
-            </collision>
-            <collision>
-                <origin xyz="0 0 0.001" rpy="0 0 0" />
-                <geometry>
-                    <cylinder radius="0.035" length="0.002" />
-                </geometry>
-            </collision>
+            <xacro:fb_tool_collision />
             <xacro:rr_inertia_cylinder_solid r="0.035" h="0.01" mass="0.25" >
                 <origin xyz="0 0 ${0.035/2}" rpy="0 0 0" />

Commit message: add bottom to watering nozzle

File: h4r_farmbot_descriptions/def/tools/watering_nozzle.xacro (robot description, xacro)
@@ -19,4 +19,20 @@
             </xacro:rr_inertia_cylinder_solid>
         </link>
+        <xacro:rr_joint_fixed parent="watering_nozzle_top" child="watering_nozzle_bottom" />
+        <link name="watering_nozzle_bottom">
+            <visual>
+                <geometry>
+                    <mesh filename="package://h4r_farmbot_descriptions/mesh/${mesh_version}/watering_nozzle_bottom.stl"/>
+                </geometry>
+            </visual>
+            <collision>
+                <geometry>
+                    <cylinder radius="0.024" length="0.0065" />
+                </geometry>
+            </collision>
+            <xacro:rr_inertia_cylinder_solid r="0.024" h="0.0065" mass="0.05" >
+                <origin xyz="0 0 0" rpy="0 0 0" />
+            </xacro:rr_inertia_cylinder_solid>
+        </link>
         <xacro:fb_utm_magnet_group name="water" parent="watering_nozzle_top" origin_z="0.0175" />
         <xacro:fb_sim_magnet name="water_magnet" parent="watering_nozzle_top" origin_z="0.005" />
