Commit message: fix utm collision

File: h4r_farmbot_descriptions/def/common/tool_collision.xacro (robot description, xacro)
@@ -5,5 +5,11 @@
        xmlns:xacro="http://ros.org/wiki/xacro" >
        <xacro:macro name="fb_tool_collision" params="origin_x:=0 origin_y:=0 origin_z:=0  origin_R:=0  origin_P:=0 origin_Y:=0">
-            <collision>
+           <collision>
+            <origin xyz="${origin_x} ${origin_y} ${origin_z+0.0135}" rpy="${origin_R} ${origin_P} ${origin_Y}" />
+                <geometry>
+                    <cylinder radius="0.033" length="0.003" />
+                </geometry>
+            </collision>
+           <collision>
                 <origin xyz="${origin_x} ${origin_y} ${origin_z+0.006}" rpy="${origin_R} ${origin_P} ${origin_Y}" />
                 <geometry>

File: h4r_farmbot_descriptions/def/farmbot/utm.xacro (robot description, xacro)
@@ -12,7 +12,7 @@
         </visual>
         <collision name="utm_col">
-            <origin xyz="0 0 0.007" rpy="0 0 0" />
+            <origin xyz="0 0 0.008" rpy="0 0 0" />
             <geometry>
-                <mesh filename="package://h4r_farmbot_descriptions/mesh/utm_collision.stl" scale="0.001 0.001 0.001" />
+                <mesh filename="package://h4r_farmbot_descriptions/mesh/utm_collision.dae" scale="0.001 0.001 0.001" />
             </geometry>
         </collision>
@@ -21,5 +21,5 @@
         </xacro:rr_inertia_cylinder_solid>
     </link>
-    <xacro:fb_sim_magnet name="magnet" parent="utm" origin_z="0.008"/>
+    <xacro:fb_sim_magnet name="magnet" parent="utm" origin_z="0.009"/>
     <!-- UTM COVER -->
     <xacro:rr_joint_fixed parent="utm" child="utm_cover" origin_z="0.051" origin_P="${-rr_const_pi}" origin_Y="${-rr_const_pi}" />
