Commit message: add test for utm and magnetic plugin - magnet seems to work in test now

File: h4r_farmbot_descriptions/def/common/magnet_group.xacro (robot description, xacro)
@@ -14,14 +14,14 @@
                origin_Y="${origin_Y}"/>
         <link name="${name}">
+            <visual name="visual">
+                <geometry>
+                    <cylinder radius="0.007" length="0.005" />
+                </geometry>
+            </visual>
             <collision name="collision">
                 <geometry>
-                    <cylinder radius="0.015" length="0.005" />
+                    <cylinder radius="0.007" length="0.005" />
                 </geometry>
             </collision>
-            <visual name="visual">
-                <geometry>
-                    <cylinder radius="0.0075" length="0.005" />
-                </geometry>
-            </visual>
         </link>
         <inertial>
@@ -30,19 +30,43 @@
             </xacro:rr_inertia_cylinder_solid>
         </inertial>
+    </xacro:macro>
+    <xacro:macro name="fb_utm_magnet_group" params="name parent origin_x:=0 origin_y:=0 origin_z:=0 origin_R:=0 origin_P:=0 origin_Y:=0" >
+        <xacro:fb_utm_magnet name="utm_magnetgroup_${name}_0" parent="${parent}" origin_x="0" origin_y= "0.0125" origin_z="${origin_z}"/>l
+        <xacro:fb_utm_magnet name="utm_magnetgroup_${name}_1" parent="${parent}" origin_x="-0.010825"  origin_y="-0.00625"  origin_z="${origin_z}"/>
+        <xacro:fb_utm_magnet name="utm_magnetgroup_${name}_2" parent="${parent}" origin_x= "0.010825"  origin_y="-0.00625"  origin_z="${origin_z}"/>
+    </xacro:macro>
+    <xacro:macro name="fb_sim_magnet" params="name parent origin_x:=0 origin_y:=0 origin_z:=0 origin_R:=0 origin_P:=0 origin_Y:=0 magnet_strength:=2" >
+        <rr_joint_fixed parent="${parent}"
+               child="${name}"
+               origin_x="${origin_x}"
+               origin_y="${origin_y}"
+               origin_z="${origin_z}"
+               origin_P="${origin_P}"
+               origin_R="${origin_R}"
+               origin_Y="${origin_Y}"/>
+        <link name="${name}">
+            <visual name="visual">
+                <geometry>
+                    <cylinder radius="0.035" length="0.005" />
+                </geometry>
+            </visual>
+            <collision name="collision">
+                <geometry>
+                    <cylinder radius="0.035" length="0.005" />
+                </geometry>
+            </collision>
+            <xacro:rr_inertia_cylinder_solid r="0.035" h="0.005" mass="0.10" >
+                <origin xyz="0 0 0" rpy="0 0 0" />
+            </xacro:rr_inertia_cylinder_solid>
+        </link>
         <gazebo>
             <plugin name="dipole_magnet" filename="libstorm_gazebo_dipole_magnet.so">
                 <bodyName>${name}</bodyName>
                 <dipole_moment>0 0 ${magnet_strength}</dipole_moment>
-                <!-- Set to false if not using ROS -->
                 <shouldPublish>false</shouldPublish>
                 <topicNs>magnet_${name}_debug</topicNs>
-                <updateRate>100</updateRate>
+                <updateRate>10</updateRate>
             </plugin>
         </gazebo>
     </xacro:macro>
-    <xacro:macro name="fb_utm_magnet_group" params="name parent origin_x:=0 origin_y:=0 origin_z:=0 origin_R:=0 origin_P:=0 origin_Y:=0 magnet_strength:=10" >
-        <xacro:fb_utm_magnet name="utm_magnetgroup_${name}_0" parent="${parent}" magnet_strength="10" origin_x="0" origin_y= "0.0125" origin_R="${rr_const_pi}" origin_z="${origin_z}"/>l
-        <xacro:fb_utm_magnet name="utm_magnetgroup_${name}_1" parent="${parent}" magnet_strength="10" origin_x="-0.010825"  origin_y="-0.00625"  origin_z="${origin_z}"/>
-        <xacro:fb_utm_magnet name="utm_magnetgroup_${name}_2" parent="${parent}" magnet_strength="10" origin_x= "0.010825"  origin_y="-0.00625"  origin_z="${origin_z}"/>
-    </xacro:macro>
 </robot>

File: h4r_farmbot_descriptions/def/farmbot/utm.xacro (robot description, xacro)
@@ -38,4 +38,13 @@
         </xacro:rr_inertia_cylinder_solid>
     </link>
-    <xacro:fb_utm_magnet_group name="utm" parent="utm" origin_z="0.0075" magnet_strength="50" />
+                <gazebo>
+            <plugin name="dipole_magnet" filename="libstorm_gazebo_dipole_magnet.so">
+                <bodyName>utm</bodyName>
+                <dipole_moment>0 0 20</dipole_moment>
+                <!-- Set to false if not using ROS -->
+                <shouldPublish>false</shouldPublish>
+                <topicNs>magnet_utm_debug</topicNs>
+                <updateRate>50</updateRate>
+            </plugin>
+        </gazebo>
 </robot>

File: h4r_farmbot_descriptions/def/test/utm_test.xacro (robot description, xacro)
@@ -7,21 +7,25 @@
         <xacro:include filename="$(find h4r_farmbot_descriptions)/def/common/magnet_group.xacro"/>
         <xacro:property name="mesh_version"            value="v1.2" />
-        <link name="watering_nozzle_top">
+        <link name="world" />
+                <rr_joint_fixed parent="world"
+               child="utm"
+               origin_z="0.4"
+                />
+        <link name="utm">
             <visual>
                 <geometry>
-                    <mesh filename="package://h4r_farmbot_descriptions/mesh/${mesh_version}/watering_nozzle_top.stl"/>
+                    <mesh filename="package://h4r_farmbot_descriptions/mesh/${mesh_version}/utm.stl"/>
                 </geometry>
             </visual>
-            <collision>
-                <origin xyz="0 0 ${0.035/4}" rpy="0 0 0" />
+            <collision name="utm_col">
+                <origin xyz="0 0 0.016" rpy="0 0 0" />
                 <geometry>
-                     <cylinder radius="0.035" length="0.016" />
+                    <mesh filename="package://h4r_farmbot_descriptions/mesh/utm_collision.stl" scale="0.001 0.001 0.001" />
                 </geometry>
             </collision>
-            <xacro:rr_inertia_cylinder_solid r="0.035" h="0.01" mass="0.25" >
-                <origin xyz="0 0 ${0.035/2}" rpy="0 0 0" />
+            <xacro:rr_inertia_cylinder_solid r="0.05" h="0.1" mass="0.25" >
+                <origin xyz="0 0 0" rpy="0 0 0" />
             </xacro:rr_inertia_cylinder_solid>
         </link>
-        <xacro:fb_utm_magnet_group name="water" parent="watering_nozzle_top" origin_z="0.0175" />
-        <xacro:fb_sim_magnet name="water_magnet" parent="watering_nozzle_top" />
+        <xacro:fb_sim_magnet name="magnet" parent="utm" origin_z="0.008"/>
 </robot>

Commit message: move current code from test into real model

File: h4r_farmbot_descriptions/def/common/magnet_group.xacro (robot description, xacro)
@@ -48,10 +48,10 @@
             <visual name="visual">
                 <geometry>
-                    <cylinder radius="0.035" length="0.005" />
+                    <cylinder radius="0.03" length="0.005" />
                 </geometry>
             </visual>
             <collision name="collision">
                 <geometry>
-                    <cylinder radius="0.035" length="0.005" />
+                    <cylinder radius="0.03" length="0.005" />
                 </geometry>
             </collision>

File: h4r_farmbot_descriptions/def/farmbot.xacro (robot description, xacro)
@@ -11,6 +11,9 @@
     <xacro:include filename="$(find h4r_farmbot_descriptions)/def/farmbot/boom.xacro"/>
     <xacro:include filename="$(find h4r_farmbot_descriptions)/def/farmbot/vertical.xacro"/>
+    <!-- UTM -->
+    <xacro:rr_joint_fixed parent="vertical" child="utm" origin_y="0.0465" origin_z="${-vertical_length/2+0.002}" origin_Y="${-rr_const_pi/2}" />
     <xacro:include filename="$(find h4r_farmbot_descriptions)/def/farmbot/utm.xacro"/>
     <xacro:include filename="$(find h4r_farmbot_descriptions)/def/farmbot/toolbays.xacro"/>
+    <xacro:include filename="$(find h4r_farmbot_descriptions)/def/common/magnet_group.xacro"/>
     <!-- ROS CONTROL PLUGIN -->
     <xacro:rr_roscontrol_controller />

File: h4r_farmbot_descriptions/def/farmbot/utm.xacro (robot description, xacro)
@@ -4,6 +4,5 @@
        xmlns:interface="http://playerstage.sourceforge.net/gazebo/xmlschema/#interface"
        xmlns:xacro="http://ros.org/wiki/xacro">
-    <xacro:include filename="$(find h4r_farmbot_descriptions)/def/common/magnet_group.xacro"/>
-    <xacro:rr_joint_fixed parent="vertical" child="utm" origin_y="0.0465" origin_z="${-vertical_length/2+0.002}" origin_Y="${-rr_const_pi/2}" />
+    <!-- UTM -->
     <link name="utm">
         <visual>
@@ -12,7 +11,8 @@
             </geometry>
         </visual>
-        <collision>
+        <collision name="utm_col">
+            <origin xyz="0 0 0.016" rpy="0 0 0" />
             <geometry>
-                <mesh filename="package://h4r_farmbot_descriptions/mesh/${mesh_version}/utm.stl"/>
+                <mesh filename="package://h4r_farmbot_descriptions/mesh/utm_collision.stl" scale="0.001 0.001 0.001" />
             </geometry>
         </collision>
@@ -21,4 +21,6 @@
         </xacro:rr_inertia_cylinder_solid>
     </link>
+    <xacro:fb_sim_magnet name="magnet" parent="utm" origin_z="0.008"/>
+    <!-- UTM COVER -->
     <xacro:rr_joint_fixed parent="utm" child="utm_cover" origin_z="0.051" origin_P="${-rr_const_pi}" origin_Y="${-rr_const_pi}" />
     <link name="utm_cover">
@@ -38,13 +40,3 @@
         </xacro:rr_inertia_cylinder_solid>
     </link>
-                <gazebo>
-            <plugin name="dipole_magnet" filename="libstorm_gazebo_dipole_magnet.so">
-                <bodyName>utm</bodyName>
-                <dipole_moment>0 0 20</dipole_moment>
-                <!-- Set to false if not using ROS -->
-                <shouldPublish>false</shouldPublish>
-                <topicNs>magnet_utm_debug</topicNs>
-                <updateRate>50</updateRate>
-            </plugin>
-        </gazebo>
 </robot>

File: h4r_farmbot_descriptions/def/test/utm_test.xacro (robot description, xacro)
@@ -8,24 +8,5 @@
         <xacro:property name="mesh_version"            value="v1.2" />
         <link name="world" />
-                <rr_joint_fixed parent="world"
-               child="utm"
-               origin_z="0.4"
-                />
-        <link name="utm">
-            <visual>
-                <geometry>
-                    <mesh filename="package://h4r_farmbot_descriptions/mesh/${mesh_version}/utm.stl"/>
-                </geometry>
-            </visual>
-            <collision name="utm_col">
-                <origin xyz="0 0 0.016" rpy="0 0 0" />
-                <geometry>
-                    <mesh filename="package://h4r_farmbot_descriptions/mesh/utm_collision.stl" scale="0.001 0.001 0.001" />
-                </geometry>
-            </collision>
-            <xacro:rr_inertia_cylinder_solid r="0.05" h="0.1" mass="0.25" >
-                <origin xyz="0 0 0" rpy="0 0 0" />
-            </xacro:rr_inertia_cylinder_solid>
-        </link>
-        <xacro:fb_sim_magnet name="magnet" parent="utm" origin_z="0.008"/>
+        <rr_joint_fixed parent="world" child="utm" origin_z="0.4" />
+       <xacro:include filename="$(find h4r_farmbot_descriptions)/def/farmbot/utm.xacro"/>
 </robot>

Commit message: shrink farmbot, and other fixes
watering nozzle magnet move up
increase magnet update rate
move toolbays to front

File: h4r_farmbot_descriptions/def/common/magnet_group.xacro (robot description, xacro)
@@ -66,5 +66,5 @@
                 <shouldPublish>false</shouldPublish>
                 <topicNs>magnet_${name}_debug</topicNs>
-                <updateRate>10</updateRate>
+                <updateRate>100</updateRate>
             </plugin>
         </gazebo>

File: h4r_farmbot_descriptions/def/farmbot.xacro (robot description, xacro)
@@ -5,4 +5,5 @@
        xmlns:xacro="http://ros.org/wiki/xacro" name="h4r_farmbot">
     <xacro:include filename="$(find h4r_rapid_robot_xacros)/def/rapid_robot.xacro"/>
+    <xacro:include filename="$(find h4r_farmbot_descriptions)/def/common/magnet_group.xacro"/>
     <xacro:include filename="$(find h4r_farmbot_descriptions)/def/farmbot/frame.xacro"/>
     <xacro:include filename="$(find h4r_farmbot_descriptions)/def/farmbot/properties.xacro"/>
@@ -15,5 +16,4 @@
     <xacro:include filename="$(find h4r_farmbot_descriptions)/def/farmbot/utm.xacro"/>
     <xacro:include filename="$(find h4r_farmbot_descriptions)/def/farmbot/toolbays.xacro"/>
-    <xacro:include filename="$(find h4r_farmbot_descriptions)/def/common/magnet_group.xacro"/>
     <!-- ROS CONTROL PLUGIN -->
     <xacro:rr_roscontrol_controller />

File: h4r_farmbot_descriptions/def/farmbot/properties.xacro (robot description, xacro)
@@ -5,6 +5,6 @@
        xmlns:xacro="http://ros.org/wiki/xacro">
     <xacro:property name="bed_height"                 value="1.0" />
-    <xacro:property name="bed_length"                 value="5.0" />
-    <xacro:property name="bed_width"                  value="2.0" />
+    <xacro:property name="bed_length"                 value="1.5" />
+    <xacro:property name="bed_width"                  value="1.0" />
     <xacro:property name="soil_height"                value="0.9" />
     <xacro:property name="wood_board_width"           value="0.04" />

File: h4r_farmbot_descriptions/def/farmbot/toolbays.xacro (robot description, xacro)
@@ -32,18 +32,20 @@
     </xacro:macro>
     <xacro:fb_toolbay
-           parent="rail_frame_3"
+           parent="rail_frame_2"
            number="0"
            mesh_version="${mesh_version}"
            origin_z="0.113"
-              origin_y="0.117"
+           origin_y="-0.117"
            origin_x="0.25"
+           origin_Y="${rr_const_pi}"
         />
     <xacro:fb_toolbay
-           parent="rail_frame_3"
+           parent="rail_frame_2"
            number="1"
            mesh_version="${mesh_version}"
            origin_z="0.113"
-              origin_y="0.117"
+           origin_y="-0.117"
            origin_x="-0.25"
+           origin_Y="${rr_const_pi}"
         />
 </robot>

File: h4r_farmbot_descriptions/def/tools/watering_nozzle.xacro (robot description, xacro)
@@ -24,4 +24,4 @@
         </link>
         <xacro:fb_utm_magnet_group name="water" parent="watering_nozzle_top" origin_z="0.0175" />
-        <xacro:fb_sim_magnet name="water_magnet" parent="watering_nozzle_top" />
+        <xacro:fb_sim_magnet name="water_magnet" parent="watering_nozzle_top" origin_z="0.005" />
 </robot>

Commit message: latest changes

File: h4r_farmbot_descriptions/def/common/magnet_group.xacro (robot description, xacro)
@@ -3,5 +3,5 @@
        xmlns:controller="http://playerstage.sourceforge.net/gazebo/xmlschema/#controller"
        xmlns:interface="http://playerstage.sourceforge.net/gazebo/xmlschema/#interface"
-       xmlns:xacro="http://ros.org/wiki/xacro" name="h4r_farmbot_tool_water">
+       xmlns:xacro="http://ros.org/wiki/xacro" >
     <xacro:macro name="fb_utm_magnet" params="name parent magnet_strength:=6 origin_x:=0 origin_y:=0 origin_z:=0  origin_R:=0  origin_P:=0 origin_Y:=0">
        <rr_joint_fixed parent="${parent}"
@@ -16,5 +16,5 @@
             <visual name="visual">
                 <geometry>
-                    <cylinder radius="0.007" length="0.005" />
+                    <cylinder radius="0.0075" length="0.005" />
                 </geometry>
             </visual>

File: h4r_farmbot_descriptions/def/farmbot/utm.xacro (robot description, xacro)
@@ -12,5 +12,5 @@
         </visual>
         <collision name="utm_col">
-            <origin xyz="0 0 0.016" rpy="0 0 0" />
+            <origin xyz="0 0 0.007" rpy="0 0 0" />
             <geometry>
                 <mesh filename="package://h4r_farmbot_descriptions/mesh/utm_collision.stl" scale="0.001 0.001 0.001" />

File: h4r_farmbot_descriptions/def/tools/watering_nozzle.xacro (robot description, xacro)
@@ -16,5 +16,5 @@
                 <origin xyz="0 0 0.006" rpy="0 0 0" />
                 <geometry>
-                    <box size="0.063 0.07 0.0074" />
+                    <box size="0.063 0.04 0.0074" />
                 </geometry>
             </collision>

Commit message: update magnets to the full radius

File: h4r_farmbot_descriptions/def/common/magnet_group.xacro (robot description, xacro)
@@ -21,5 +21,5 @@
             <collision name="collision">
                 <geometry>
-                    <cylinder radius="0.007" length="0.005" />
+                    <cylinder radius="0.0075" length="0.005" />
                 </geometry>
             </collision>

Commit message: change magnet strengths

File: h4r_farmbot_descriptions/def/common/magnet_group.xacro (robot description, xacro)
@@ -36,5 +36,5 @@
         <xacro:fb_utm_magnet name="utm_magnetgroup_${name}_2" parent="${parent}" origin_x= "0.010825"  origin_y="-0.00625"  origin_z="${origin_z}"/>
     </xacro:macro>
-    <xacro:macro name="fb_sim_magnet" params="name parent origin_x:=0 origin_y:=0 origin_z:=0 origin_R:=0 origin_P:=0 origin_Y:=0 magnet_strength:=2" >
+    <xacro:macro name="fb_sim_magnet" params="name parent origin_x:=0 origin_y:=0 origin_z:=0 origin_R:=0 origin_P:=0 origin_Y:=0 magnet_strength:=3" >
         <rr_joint_fixed parent="${parent}"
                child="${name}"

File: h4r_farmbot_descriptions/def/farmbot/utm.xacro (robot description, xacro)
@@ -21,5 +21,5 @@
         </xacro:rr_inertia_cylinder_solid>
     </link>
-    <xacro:fb_sim_magnet name="magnet" parent="utm" origin_z="0.009"/>
+    <xacro:fb_sim_magnet name="magnet" parent="utm" origin_z="0.009" magnet_strength="6" />
     <!-- UTM COVER -->
     <xacro:rr_joint_fixed parent="utm" child="utm_cover" origin_z="0.051" origin_P="${-rr_const_pi}" origin_Y="${-rr_const_pi}" />
